Commit message: new ajusts and files

File: vrx_urdf/wamv_gazebo/urdf/dynamics/wamv_gazebo_dynamics_plugin.xacro (robot description, xacro)
@@ -16,7 +16,4 @@
           <point>-1.4 1.03 0</point>
         </points>
-        <wavefield>
-          <topic>/vrx/wavefield/parameters</topic>
-        </wavefield>
       </plugin>
       <!-- Right hull -->
@@ -32,28 +29,29 @@
           <point>-1.4 -1.03 0</point>
         </points>
-        <wavefield>
-          <topic>/vrx/wavefield/parameters</topic>
-        </wavefield>
       </plugin>
       <plugin
-        filename="libSimpleHydrodynamics.so"
-        name="vrx::SimpleHydrodynamics">
-        <link_name>${namespace}/base_link</link_name>
-        <!-- Added mass -->
-        <xDotU>0.0</xDotU>
-        <yDotV>0.0</yDotV>
-        <nDotR>0.0</nDotR>
-        <!-- Linear and quadratic drag -->
-        <xU>100.0</xU>
-        <xUU>150.0</xUU>
-        <yV>100.0</yV>
-        <yVV>100.0</yVV>
-        <zW>500.0</zW>
-        <kP>300.0</kP>
-        <kPP>600.0</kPP>
-        <mQ>900.0</mQ>
-        <mQQ>900.0</mQQ>
-        <nR>800.0</nR>
-        <nRR>800.0</nRR>
+        filename="gz-waves1-hydrodynamics-system"
+        name="gz::sim::systems::Hydrodynamics">
+        <!-- Or apply hydrodynamics to named links -->
+        <enable>${namespace}::base_link</enable>
+        <!-- Hydrodynamics -->
+        <hydrodynamics>
+          <damping_on>1</damping_on>
+          <viscous_drag_on>1</viscous_drag_on>
+          <pressure_drag_on>1</pressure_drag_on>
+          <!-- Linear and Angular Damping -->
+          <cDampL1>1.0E-6</cDampL1>
+          <cDampL2>1.0E-6</cDampL2>
+          <cDampR1>1.0E-6</cDampR1>
+          <cDampR2>1.0E-6</cDampR2>
+          <!-- 'Pressure' Drag -->
+          <cPDrag1>1.0E+2</cPDrag1>
+          <cPDrag2>1.0E+2</cPDrag2>
+          <fPDrag>0.4</fPDrag>
+          <cSDrag1>1.0E+2</cSDrag1>
+          <cSDrag2>1.0E+2</cSDrag2>
+          <fSDrag>0.4</fSDrag>
+          <vRDrag>1.0</vRDrag>
+        </hydrodynamics>
       </plugin>
     </gazebo>

File: vrx_urdf/wamv_gazebo/urdf/wamv_gazebo.urdf.xacro (robot description, xacro)
@@ -3,4 +3,7 @@
 <robot xmlns:xacro="http://ros.org/wiki/xacro"
        name="WAM-V">
+  <!-- Parâmetro global de escala para o WAMV -->
+  <xacro:arg name="wamv_scale" default="0.5" />
+  <xacro:property name="wamv_scale" value="$(arg wamv_scale)" scope="global" />
   <xacro:arg name="locked" default="false" />
   <xacro:arg name="thruster_config" default="H" />
@@ -36,7 +39,4 @@
   <xacro:include filename="$(find wamv_gazebo)/urdf/wamv_gazebo.xacro"/>
   <!-- === Batteries === -->
-  <xacro:include filename="$(find wamv_description)/urdf/battery.xacro"/>
-  <xacro:battery prefix="left" position="0 1 0.45" orientation="0 0 0"/>
-  <xacro:battery prefix="right" position="0 -1 0.45" orientation="0 0 0"/>
   <!-- === Thrusters === -->
   <!-- Use thruster yaml file if given -->
@@ -95,14 +95,12 @@
     <xacro:include filename="$(arg component_xacro_file)"/>
     <xacro:yaml_components />
-    <!-- Add CPU Cases -->
-    <xacro:include filename="$(find wamv_description)/urdf/cpu_cases.xacro" />
-    <xacro:cpu_cases position="-0.15 0 1.53" orientation="0 0 0"/>
   </xacro:if>
   <!-- Otherwise, add sensors based on enable variables -->
   <xacro:unless value="$(arg yaml_component_generation)">
     <!-- Add a front camera -->
-    <xacro:if value="$(arg camera_enabled)">
-      <xacro:wamv_camera name="front_camera" y="0.3" x="0.75" P="${radians(15)}" />
-    </xacro:if>
+    <xacro:wamv_camera name="right_camera" y="-0.45" x="0" P="${radians(30)}" Y="${radians(-90)}" post_Y="${radians(-90)}" />
+    <xacro:wamv_camera name="left_camera" y="0.45" x="0" P="${radians(30)}" Y="${radians(90)}" post_Y="${radians(90)}" />
+    <xacro:wamv_camera name="front_camera" y="0" x="0.85" P="${radians(30)}" Y="${radians(0)}" post_Y="${radians(0)}" />
+    <xacro:wamv_camera name="back_camera" y="0" x="-0.85" P="${radians(30)}" Y="${radians(-180)}" post_Y="${radians(-180)}" />
     <!-- Add simulated GPS -->
     <xacro:if value="$(arg gps_enabled)">
@@ -113,40 +111,18 @@
       <xacro:wamv_imu name="imu_wamv" y="-0.2" />
     </xacro:if>
-    <!-- Add 3D LIDAR -->
-    <xacro:if value="$(arg lidar_enabled)">
-      <xacro:lidar name="lidar_wamv" y="-0.3" type="16_beam"/>
-    </xacro:if>
     <!-- Add P3D ground truth -->
     <xacro:if value="$(arg ground_truth_enabled)">
       <xacro:wamv_p3d name="p3d_wamv"/>
     </xacro:if>
-    <!-- Add pinger -->
-    <xacro:if value="$(arg pinger_enabled)">
-      <xacro:wamv_pinger sensor_name="receiver" position="-528 191 -2.0" />
-    </xacro:if>
-    <!-- Add ball shooter (default pitch angle: ~-60 deg) -->
-    <xacro:if value="$(arg ball_shooter_enabled)">
-      <xacro:wamv_ball_shooter name="ball_shooter" x="0.54" y="0.30" z="1.296" pitch="-1.04"/>
-    </xacro:if>
     <!-- ==== VRX sensor configuration ==== -->
     <xacro:if value="$(arg vrx_sensors_enabled)">
       <!-- Add CPU Cases -->
-      <xacro:include filename="$(find wamv_description)/urdf/cpu_cases.xacro" />
-      <xacro:cpu_cases position="-0.15 0 1.53" orientation="0 0 0"/>
-      <!-- Add a stereo camera pair -->
-      <xacro:wamv_camera name="front_left_camera" y="0.1" x="0.75" P="${radians(15)}" />
-      <xacro:wamv_camera name="front_right_camera" y="-0.1" x="0.75" P="${radians(15)}" />
-      <!-- Add a camera facing right -->
-      <xacro:wamv_camera name="middle_right_camera" y="-0.45" P="${radians(15)}" Y="${radians(-90)}" post_Y="${radians(-90)}" />
+      <!-- Add Containment Boom -->
+      <xacro:include filename="$(find wamv_description)/urdf/boom.xacro" />
+      <xacro:containment_boom position="2.6 0 2" orientation="0 0 ${radians(90)}"/>
       <!-- Add simulated GPS -->
-      <xacro:wamv_gps name="gps_wamv" x="-0.85" />
+      <xacro:wamv_gps name="gps_wamv" x="0" />
       <!-- Add Simulated IMU -->
       <xacro:wamv_imu name="imu_wamv" y="-0.2" />
-      <!-- Add 3D LIDAR -->
-      <xacro:lidar name="lidar_wamv" type="16_beam"/>
-      <!-- Add pinger -->
-      <xacro:wamv_pinger sensor_name="receiver" position="-528 191 -2.0" />
-      <!-- Add ball shooter (default pitch angle: ~-60 deg) -->
-      <xacro:wamv_ball_shooter name="ball_shooter" x="0.54" y="0.30" z="1.296" pitch="-1.04"/>
     </xacro:if>
   </xacro:unless>
